File: navspark_rpi_shield.sch (KiCad schematic (older format))
At the start: 5 parts, among them P1 CONN_02X13, P2 CONN_01X13, P3 CONN_01X12

Commit message: small changes
Changed lines of the file:
@@
 Text Label 3300 2650 0    60   ~ 0
 GND
-Text Label 2650 3050 2    60   ~ 0
+Text Label 2800 3050 2    60   ~ 0
 5V
 $Comp
@@
 NoConn ~ 3300 3050
 NoConn ~ 3300 2250
-Text Label 3550 1850 0    60   ~ 0
+Text Label 3300 1850 0    60   ~ 0
 GND
-Wire Wire Line
-	3300 1850 3550 1850
-Wire Wire Line
-	2800 3050 2650 3050
 Text Label 5450 2450 2    60   ~ 0
 SPI_MOSI

Commit message: save changes before submission
Other:
- note added: "Note: \nthe pin numbering here does\nnot directly correspond to the\nRPi pin numbers, to account\nfor the connector's header\norientation."
- note removed: "(note: the pin numbering here does not correspond to\nthe Raspberry pin numbers, to account for the header\norientation)"
Changed lines of the file:
@@
 P 5650 2450
 F 0 "P2" H 5650 3150 50  0000 C CNN
-F 1 "CONN_01X13" V 5750 2450 50  0000 C CNN
+F 1 "CONN_01X13" V 5750 2500 50  0000 C CNN
 F 2 "Pin_Headers:Pin_Header_Straight_1x13" H 5650 2450 50  0001 C CNN
 F 3 "" H 5650 2450 50  0000 C CNN
@@
 	1    0    0    -1
 $EndComp
-Wire Wire Line
-	4400 2150 4400 2300
-Wire Wire Line
-	4400 2600 4400 2750
 Text Label 4100 2250 2    60   ~ 0
 5V
@@
 NoConn ~ 2800 2050
 NoConn ~ 6200 2750
-Connection ~ 4400 2250
-Connection ~ 4400 2650
-Text Notes 2250 3650 0    60   Italic 0
-(note: the pin numbering here does not correspond to\nthe Raspberry pin numbers, to account for the header\norientation)
+Text Notes 2400 3900 0    60   Italic 0
+Note: \nthe pin numbering here does\nnot directly correspond to the\nRPi pin numbers, to account\nfor the connector's header\norientation.
 $Comp
 L C C2
@@
 	1    0    0    -1
 $EndComp
-Wire Wire Line
-	4650 2200 4650 2300
-Wire Wire Line
-	4650 2600 4650 2700
-Wire Wire Line
-	4100 2250 4400 2250
-Wire Wire Line
-	4400 2200 4650 2200
-Connection ~ 4400 2200
-Wire Wire Line
-	4650 2700 4400 2700
 $Comp
 L GND #PWR04
@@
 	1    0    0    -1
 $EndComp
-Connection ~ 4400 2700
-Wire Wire Line
-	4100 2650 4400 2650
 Text Notes 5100 3800 0    60   Italic 0
 Regular sizeboards, at the moment:\n* NavSpark\n* NavSpark-GL\n* NavSpark-BD\nand other compatible boards
+Wire Wire Line
+	4400 2150 4400 2300
+Wire Wire Line
+	4400 2600 4400 2750
+Connection ~ 4400 2250
+Connection ~ 4400 2650
+Wire Wire Line
+	4650 2200 4650 2300
+Wire Wire Line
+	4650 2600 4650 2700
+Wire Wire Line
+	4100 2250 4400 2250
+Wire Wire Line
+	4400 2200 4650 2200
+Connection ~ 4400 2200
+Wire Wire Line
+	4650 2700 4400 2700
+Connection ~ 4400 2700
+Wire Wire Line
+	4100 2650 4400 2650
 $EndSCHEMATC

Commit message: add v2 of the board
Parts:
- P1: value CONN_02X13 -> RPI_02X13; footprint Pin_Headers:Pin_Header_Straight_2x13 -> Socket_Strips:Socket_Strip_Straight_2x13
- P2: value CONN_01X13 -> NAV_01X13; footprint Pin_Headers:Pin_Header_Straight_1x13 -> Socket_Strips:Socket_Strip_Straight_1x13
- P3: value CONN_01X12 -> NAV_01X12; footprint Pin_Headers:Pin_Header_Straight_1x12 -> Socket_Strips:Socket_Strip_Straight_1x12
Connections:
- net 1PPS: now also P1.26 (P26); no longer P1.16 (P16)
- net GND: now also P1.14 (P14), P1.20 (P20), P1.25 (P25), P1.6 (P6), P1.9 (P9); no longer P1.10 (P10), P1.13 (P13), P1.19 (P19), P1.26 (P26), P1.5 (P5), P3.1 (P1)
- net GPIO12: now also P1.11 (P11); no longer P1.12 (P12)
- net GPIO13: now also P1.13 (P13); no longer P1.11 (P11)
- net GPIO14: now also P1.18 (P18); no longer P1.14 (P14)
- net GPIO16: now also P1.12 (P12); no longer P1.15 (P15)
- net GPIO20: now also P1.16 (P16); no longer P1.17 (P17)
- net I2C_SCL: now also P1.5 (P5); no longer P1.6 (P6)
- net I2C_SDA: now also P1.3 (P3); no longer P1.4 (P4)
- net N_TXD1: now also P1.10 (P10); no longer P1.9 (P9)
- net SPI_CSN0: now also P1.24 (P24); no longer P1.23 (P23)
- net SPI_MISO: now also P1.21 (P21); no longer P1.22 (P22)
- net SPI_MOSI: now also P1.19 (P19); no longer P1.20 (P20)
- net SPI_SCK: now also P1.23 (P23); no longer P1.24 (P24)
- net TRIG: now also P1.7 (P7); no longer P1.8 (P8)
- net VCC: now also P1.2 (P2); no longer P1.1 (P1)
- no-connect marks 14 -> 15
Other:
- note added: "Supporting regular size NavSpark boards,\nat the moment:\n* NavSpark\n* NavSpark-GL\n* NavSpark-BD\nand other compatible pinouts"
- note removed: "Note: \nthe pin numbering here does\nnot directly correspond to the\nRPi pin numbers, to account\nfor the connector's header\norientation."
- note removed: "Regular sizeboards, at the moment:\n* NavSpark\n* NavSpark-GL\n* NavSpark-BD\nand other compatible boards"
Changed lines of the file:
@@
 Sheet 1 1
 Title "NavSpark Shield for Raspberry Pi"
-Date "2015-12-20"
-Rev "v1"
+Date "2016-01-14"
+Rev "v2"
 Comp "Moonpunch"
 Comment1 "CERN Open Hardware License 1.2"
@@
 P 3050 2450
 F 0 "P1" H 3050 3150 50  0000 C CNN
-F 1 "CONN_02X13" V 3050 2450 50  0000 C CNN
-F 2 "Pin_Headers:Pin_Header_Straight_2x13" H 3050 1700 50  0001 C CNN
+F 1 "RPI_02X13" V 3050 2450 50  0000 C CNN
+F 2 "Socket_Strips:Socket_Strip_Straight_2x13" H 3050 1700 50  0001 C CNN
 F 3 "" H 3050 1300 50  0000 C CNN
 	1    3050 2450
-	1    0    0    1
+	-1   0    0    1
 $EndComp
 $Comp
@@
 P 5650 2450
 F 0 "P2" H 5650 3150 50  0000 C CNN
-F 1 "CONN_01X13" V 5750 2500 50  0000 C CNN
-F 2 "Pin_Headers:Pin_Header_Straight_1x13" H 5650 2450 50  0001 C CNN
+F 1 "NAV_01X13" V 5750 2500 50  0000 C CNN
+F 2 "Socket_Strips:Socket_Strip_Straight_1x13" H 5650 2450 50  0001 C CNN
 F 3 "" H 5650 2450 50  0000 C CNN
 	1    5650 2450
@@
 P 6000 2500
 F 0 "P3" H 6000 3150 50  0000 C CNN
-F 1 "CONN_01X12" V 6100 2500 50  0000 C CNN
-F 2 "Pin_Headers:Pin_Header_Straight_1x12" H 6000 2500 50  0001 C CNN
+F 1 "NAV_01X12" V 6100 2500 50  0000 C CNN
+F 2 "Socket_Strips:Socket_Strip_Straight_1x12" H 6000 2500 50  0001 C CNN
 F 3 "" H 6000 2500 50  0000 C CNN
 	1    6000 2500
@@
 Text Label 2800 1950 2    60   ~ 0
 SPI_CSN0
-NoConn ~ 2800 1850
-Text Label 3300 2350 0    60   ~ 0
+NoConn ~ 3300 2350
+Text Label 2800 1850 2    60   ~ 0
 1PPS
 Text Label 3300 1950 0    60   ~ 0
@@
 GND
 Text Label 2800 2450 2    60   ~ 0
-GND
-Text Label 6200 3050 0    60   ~ 0
 GND
 NoConn ~ 6200 2950
@@
 Text Label 5450 2950 2    60   ~ 0
 GPIO16
-Text Label 2800 2350 2    60   ~ 0
+Text Label 2800 2550 2    60   ~ 0
 GPIO16
 Text Label 5450 2850 2    60   ~ 0
 GPIO20
-Text Label 2800 2250 2    60   ~ 0
+Text Label 2800 2350 2    60   ~ 0
 GPIO20
 NoConn ~ 5450 2650
 Text Label 5450 2250 2    60   ~ 0
 GPIO14
-Text Label 3300 2450 0    60   ~ 0
+Text Label 2800 2250 2    60   ~ 0
 GPIO14
 Text Label 6200 2650 0    60   ~ 0
@@
 Text Label 3300 2550 0    60   ~ 0
 GPIO12
-Text Label 2800 2550 2    60   ~ 0
+Text Label 3300 2450 0    60   ~ 0
 GPIO13
 NoConn ~ 2800 2050
 NoConn ~ 6200 2750
-Text Notes 2400 3900 0    60   Italic 0
-Note: \nthe pin numbering here does\nnot directly correspond to the\nRPi pin numbers, to account\nfor the connector's header\norientation.
 $Comp
 L C C2
@@
 $EndComp
 Text Notes 5100 3800 0    60   Italic 0
-Regular sizeboards, at the moment:\n* NavSpark\n* NavSpark-GL\n* NavSpark-BD\nand other compatible boards
+Supporting regular size NavSpark boards,\nat the moment:\n* NavSpark\n* NavSpark-GL\n* NavSpark-BD\nand other compatible pinouts
 Wire Wire Line
 	4400 2150 4400 2300
@@
 Wire Wire Line
 	4100 2650 4400 2650
+NoConn ~ 6200 3050
 $EndSCHEMATC
